File: stmsplat2.sch (KiCad schematic (older format))
At the start: 115 parts, among them J1 C11_2X36, J10 Conn_01x03_Male, J11 Conn_01x02_Male, J12 Conn_01x04_Male, J13 Conn_01x04_Male, J14 Conn_01x02, J15 Conn_01x02, J16 Screw_Terminal_01x03, J17 Screw_Terminal_01x02, J18 Conn_01x02_Male, J19 Conn_01x02_Male, J2 C12_2X36, J3 Conn_01x04_Male, J4 Conn_01x04_Male, J5 Conn_Coaxial, J6 Conn_01x04_Male, J7 Conn_01x04_Male, J8 Conn_01x04_Male, J9 Conn_01x03_Male, Q1 BSS138LT1G, SW1 SW_DIP_x02, U1 ublox_chinese_PCB_module, U10 XCVR_E30-400M20S (Si4463), U11 3115_module, U2 ESP-C3-13U, U3 SST25VF032B, U4 48L512-48LM01, U5 Opamp_Quad_MCP6024, U6 E180-ZG120A, U7 AZ1084C, U8 MCP6S93-X_UN, U9 DS2485

Commit message: Splat2 Revision A.  Work-in-progress
Parts:
- J1, J2: footprint Connector_Samtec_HLE_THT:Samtec_HLE-136-02-xx-DV-TE_2x36_P2.54mm_Horizontal -> Connector_PinSocket_2.54mm:PinSocket_2x36_P2.54mm_Vertical
- R7, R8: value 4K7 -> 1K
Connections:
- net +3V3: now also C1.1, C14.2, C15.1, C16.2, C17.2, C18.1, C19.2, C2.1, C20.1, C21.2, C28.1, C3.1, C30.1, C31.1, FB2.1, J12.1 (Pin_1), J13.1 (Pin_1), J19.2 (Pin_2), J4.1 (Pin_1), J7.1 (Pin_1), Q1.3 (D), R1.1, R11.1, R13.1, R14.1, R16.2, R21.1, R22.1, R4.1, U1.1 (VCC), U10.9 (VCC), U11.5 (Pin_5), U2.1 (3V3), U3.8 (VDD), U4.8 (VCC), U6.3 (VCC), U9.6 (VCC)
- net +5V: no longer C11.1, FB1.2, J1.18 (Pin_18), J1.6 (Pin_6), U7.3 (VI)
- net GNDA: no longer R10.2
- net HALF3V3: now also R10.2
- net PB9: no longer U11.1 (Pin_1)
- net PD0: now also U11.1 (Pin_1)
- net OUR3V3: now reaches C13.1, C24.1, J16.2 (Pin_2), J19.1 (Pin_1), U7.2 (VO)
- removed net VDD: C1.1, C14.2, C15.1, C16.2, C17.2, C18.1, C19.2, C2.1, C20.1, C21.2, C28.1, C3.1, C30.1, C31.1, FB2.1, J1.5 (Pin_5), J12.1 (Pin_1), J13.1 (Pin_1), J19.2 (Pin_2), J4.1 (Pin_1), J7.1 (Pin_1), Q1.3 (D), R1.1, R11.1, R13.1, R14.1, R16.2, R21.1, R22.1, R4.1, U1.1 (VCC), U10.9 (VCC), U11.5 (Pin_5), U2.1 (3V3), U3.8 (VDD), U4.8 (VCC), U6.3 (VCC), U9.6 (VCC)
- new net +5VSTM: J1.18 (Pin_18)
- new net 3V3_VPP: J1.5 (Pin_5)
- new net 5VEXT: C11.1, FB1.2, J1.6 (Pin_6), U7.3 (VI)
- no-connect marks 71 -> 70
Other:
- note added: "PIN1 +5V PSU INPUT\nPIN2 +3V3 OUTPUT\nPIN3 GROUND\n\n"
- note added: "VER 0.20\nStart Splat2 Rev A: Fixes from prototype PCB"
- note removed: "PIN3 GROUND\nPIN2 +3V3 OUTPUT\nPIN1 +5V PSU INPUT"
- note removed: "VER 0.18\nPOWERCONN REASSIGN PINOUT"
- moved on the sheet: C10
Changed lines of the file:
@@
 GND
 Text GLabel 900  9250 0    50   Input ~ 0
-VDD
++3V3
 Wire Wire Line
 	12700 3050 12450 3050
@@
 Wire Wire Line
 	12700 8750 12700 8950
-Wire Wire Line
-	13950 8500 14300 8500
 Connection ~ 14300 8500
 $Comp
@@
 	15600 2300 15350 2300
 Text GLabel 13250 900  0    50   Input ~ 0
-VDD
++3V3
 $Comp
 L Device:LED D9
@@
 Text GLabel 4000 6400 0    50   Input ~ 0
 PG9
-$Comp
-L power:GND #PWR02
-U 1 1 5C061845
-P 4350 8500
-F 0 "#PWR02" H 4350 8250 50  0001 C CNN
-F 1 "GND" H 4355 8327 50  0000 C CNN
-F 2 "" H 4350 8500 50  0001 C CNN
-F 3 "" H 4350 8500 50  0001 C CNN
-	1    4350 8500
-	1    0    0    -1
-$EndComp
 Text GLabel 4000 6600 0    50   Input ~ 0
 PG15
@@
 $EndComp
 Text GLabel 11700 7300 1    50   Input ~ 0
-VDD
++3V3
 $Comp
 L Device:R R6
@@
 	1250 7750 1600 7750
 Text GLabel 1600 7450 2    50   Input ~ 0
-VDD
++3V3
 Text GLabel 1600 7550 2    50   Input ~ 0
 PD6
@@
 	15650 6650 15650 6750
 Text GLabel 15650 6650 1    50   Input ~ 0
-VDD
++3V3
 $Comp
 L Device:Q_PMOS_SGD Q1
@@
 Connection ~ 10750 9450
 Text GLabel 7400 3550 1    50   Input ~ 0
-VDD
++3V3
 Wire Wire Line
 	9400 10150 9400 9900
@@
 IOREF
 Text GLabel 1650 1800 2    50   Input ~ 0
-+5V
++5VSTM
 Text GLabel 1650 1900 2    50   Input ~ 0
 GND
@@
 Text GLabel 1150 1100 0    50   Input ~ 0
 PC12
-Text GLabel 1150 1200 0    50   Input ~ 0
-VDD
 Text Label 1150 1300 2    50   ~ 0
 BOOT0
@@
 Text GLabel 1150 3700 0    50   Input ~ 0
 PD1
-Text Label 1150 3800 2    50   ~ 0
-PD0
 Text GLabel 1150 3900 0    50   Input ~ 0
 PG0
@@
 F 0 "J1" H 1400 4617 50  0000 C CNN
 F 1 "C11_2X36" H 1400 4526 50  0000 C CNN
-F 2 "Connector_Samtec_HLE_THT:Samtec_HLE-136-02-xx-DV-TE_2x36_P2.54mm_Horizontal" H 1350 2700 50  0001 C CNN
+F 2 "Connector_PinSocket_2.54mm:PinSocket_2x36_P2.54mm_Vertical" H 1350 2700 50  0001 C CNN
 F 3 "~" H 1350 2700 50  0001 C CNN
 	1    1350 2700
@@
 F 0 "J2" H 2750 4617 50  0000 C CNN
 F 1 "C12_2X36" H 2750 4526 50  0000 C CNN
-F 2 "Connector_Samtec_HLE_THT:Samtec_HLE-136-02-xx-DV-TE_2x36_P2.54mm_Horizontal" H 2700 2700 50  0001 C CNN
+F 2 "Connector_PinSocket_2.54mm:PinSocket_2x36_P2.54mm_Vertical" H 2700 2700 50  0001 C CNN
 F 3 "~" H 2700 2700 50  0001 C CNN
 	1    2700 2700
@@
 	3950 7950 3950 8500
 Wire Wire Line
-	3550 8500 3950 8500
+	3550 8500 3750 8500
 Wire Wire Line
 	4250 7600 4250 8050
@@
 	3850 7200 4450 7200
 Text GLabel 4050 7000 2    50   Input ~ 0
-VDD
++3V3
 Text Notes 5000 10050 0    50   ~ 0
 RX
@@
 $EndComp
 Text GLabel 12100 3850 1    50   Input ~ 0
-VDD
++3V3
 Wire Wire Line
 	11950 4300 12100 4300
@@
 	9600 3950 9600 4200
 Text GLabel 9950 3450 1    50   Input ~ 0
-VDD
++3V3
 Wire Wire Line
 	9950 3650 9950 3450
@@
 $EndComp
 Text GLabel 8350 5800 2    50   Input ~ 0
-VDD
++3V3
 Wire Wire Line
 	7850 6950 7950 6950
@@
 	12950 6200 13450 6200
 Wire Wire Line
-	13000 6100 13450 6100
-Wire Wire Line
 	12950 6000 13450 6000
 Text GLabel 12950 5900 0    50   Input ~ 0
@@
 	15800 5550 15800 5650
 Text GLabel 15800 5550 1    50   Input ~ 0
-VDD
++3V3
 Wire Wire Line
 	15250 6100 15400 6100
@@
 Connection ~ 3400 10900
 Wire Wire Line
-	4350 8250 4350 8500
-Connection ~ 9900 2650
-Wire Wire Line
 	14350 3550 15450 3550
 $Comp
@@
 	11850 2550 11850 2650
 Wire Wire Line
-	10750 2650 10750 3350
-Wire Wire Line
-	10750 3350 11850 3350
-Wire Wire Line
-	9900 2650 10750 2650
-Wire Wire Line
 	11850 2550 12150 2550
 Wire Wire Line
@@
 P 10550 950
 F 0 "R7" H 10620 996 50  0000 L CNN
-F 1 "4K7" H 10620 905 50  0000 L CNN
+F 1 "1K" H 10620 905 50  0000 L CNN
 F 2 "Resistor_SMD:R_0805_2012Metric" V 10480 950 50  0001 C CNN
 F 3 "~" H 10550 950 50  0001 C CNN
@@
 P 10550 1450
 F 0 "R8" H 10620 1496 50  0000 L CNN
-F 1 "4K7" H 10620 1405 50  0000 L CNN
+F 1 "1K" H 10620 1405 50  0000 L CNN
 F 2 "Resistor_SMD:R_0805_2012Metric" V 10480 1450 50  0001 C CNN
 F 3 "~" H 10550 1450 50  0001 C CNN
@@
 Wire Wire Line
 	12700 3150 12550 3150
-Wire Wire Line
-	12550 3350 11850 3350
-Connection ~ 11850 3350
 $Comp
 L Connector:Conn_01x02_Male J11
@@
 $EndComp
 Wire Wire Line
-	10200 7650 10300 7650
-Wire Wire Line
 	10000 8150 9800 8150
 Wire Wire Line
-	10000 9450 10300 9450
-Wire Wire Line
 	900  9250 1000 9250
 Wire Wire Line
@@
 	1000 9250 1350 9250
 $Comp
-L Device:C C10
-U 1 1 6207CE49
-P 10300 9200
-F 0 "C10" H 10415 9246 50  0000 L CNN
-F 1 "0.1uF" H 10415 9155 50  0000 L CNN
-F 2 "Capacitor_SMD:C_0805_2012Metric" H 10338 9050 50  0001 C CNN
-F 3 "~" H 10300 9200 50  0001 C CNN
-	1    10300 9200
-	1    0    0    -1
-$EndComp
-Wire Wire Line
-	10300 9050 10300 7650
-Connection ~ 10300 7650
-Wire Wire Line
-	10300 9350 10300 9450
-Connection ~ 10300 9450
-Wire Wire Line
-	10300 9450 10750 9450
-$Comp
 L Device:C C9
 U 1 1 62109AB0
@@
 	6000 10500 5800 10500
 Text GLabel 5800 10500 0    50   Input ~ 0
-VDD
++3V3
 Text Notes 5600 10400 0    50   ~ 0
 I2C1_SCL
@@
 	5600 10200 6000 10200
 Text GLabel 5600 10100 0    50   Input ~ 0
-PB9
+PD0
 Text Notes 5600 10100 0    50   ~ 0
 INT2
@@
 SERIAL FLASH ROM\n  AND NVRAM
 Text Notes 12400 10400 0    89   Italic 0
-VER 0.18\nPOWERCONN REASSIGN PINOUT
+VER 0.20\nStart Splat2 Rev A: Fixes from prototype PCB
 $Comp
 L Connector_Generic:Conn_01x02 J14
@@
 	12300 7950 12700 7950
 Text GLabel 13500 8750 2    50   Input ~ 0
-VDD
++3V3
 $Comp
 L Connector:Screw_Terminal_01x03 J16
@@
 	-1   0    0    -1
 $EndComp
-Text Notes 8100 7950 0    50   ~ 0
-PIN3 GROUND\nPIN2 +3V3 OUTPUT\nPIN1 +5V PSU INPUT
-Wire Wire Line
-	10300 7650 10550 7650
+Text Notes 8100 8050 0    50   ~ 0
+PIN1 +5V PSU INPUT\nPIN2 +3V3 OUTPUT\nPIN3 GROUND\n\n
 $Comp
 L Connector:Conn_01x04_Male J13
@@
 	1250 8550 1600 8550
 Text GLabel 1600 8450 2    50   Input ~ 0
-VDD
++3V3
 Text Label 1600 8550 0    50   ~ 0
 PF6
@@
 Connection ~ 13300 7950
 Wire Wire Line
-	13300 7950 14750 7950
-Wire Wire Line
 	13000 7950 13300 7950
 NoConn ~ 2500 1300
@@
 NoConn ~ 2500 2000
 NoConn ~ 2500 2100
-NoConn ~ 1650 1700
 NoConn ~ 1650 2100
 NoConn ~ 1150 1300
@@
 NoConn ~ 1650 2700
 NoConn ~ 1150 2900
-NoConn ~ 1150 3800
 NoConn ~ 1650 3600
 NoConn ~ 1650 4300
@@
 $EndComp
 Text GLabel 10950 7650 2    50   Input ~ 0
-+5V
+5VEXT
 Text GLabel 1650 1200 2    50   Input ~ 0
-+5V
+5VEXT
 $Comp
 L power:PWR_FLAG #FLG0101
@@
 Wire Wire Line
 	3250 2500 3000 2500
-Connection ~ 12550 3350
 Wire Wire Line
 	12550 3150 12550 3350
@@
 Text GLabel 1650 1600 2    50   Input ~ 0
 NRST
-Text Label 1650 1700 0    50   ~ 0
-+3V3
 NoConn ~ 1650 1500
 Text GLabel 4200 2050 2    50   Input ~ 0
@@
 Wire Wire Line
 	3850 3800 3850 4000
+Wire Wire Line
+	12950 6100 13450 6100
+Wire Wire Line
+	12450 3050 12450 3450
+Wire Wire Line
+	12450 3450 11850 3450
+Wire Wire Line
+	11850 3450 11850 3350
+Connection ~ 12450 3050
+Wire Wire Line
+	10200 7650 10550 7650
+Wire Wire Line
+	10000 9450 10750 9450
+Wire Wire Line
+	13950 8500 14300 8500
+Wire Wire Line
+	13300 7950 14750 7950
+$Comp
+L Device:C C10
+U 1 1 6207CE49
+P 3750 8650
+F 0 "C10" H 3865 8696 50  0000 L CNN
+F 1 "0.1uF" H 3865 8605 50  0000 L CNN
+F 2 "Capacitor_SMD:C_0805_2012Metric" H 3788 8500 50  0001 C CNN
+F 3 "~" H 3750 8650 50  0001 C CNN
+	1    3750 8650
+	1    0    0    -1
+$EndComp
+Connection ~ 3750 8500
+Wire Wire Line
+	3750 8500 3950 8500
+$Comp
+L power:GND #PWR0113
+U 1 1 621EFDA2
+P 3750 8850
+F 0 "#PWR0113" H 3750 8600 50  0001 C CNN
+F 1 "GND" H 3755 8677 50  0000 C CNN
+F 2 "" H 3750 8850 50  0001 C CNN
+F 3 "" H 3750 8850 50  0001 C CNN
+	1    3750 8850
+	1    0    0    -1
+$EndComp
+Wire Wire Line
+	3750 8850 3750 8800
+Wire Wire Line
+	3750 8800 4350 8800
+Connection ~ 3750 8800
+Wire Wire Line
+	4350 8250 4350 8800
+Text GLabel 1650 1700 2    50   Input ~ 0
++3V3
+Text Label 1150 1200 2    50   ~ 0
+3V3_VPP
+NoConn ~ 1150 1200
+Text Label 11200 7850 0    50   ~ 0
+OUR3V3
+Text GLabel 1150 3800 0    50   Input ~ 0
+PD0
 $EndSCHEMATC

Commit message: Routed but needs checking
Parts:
- removed J9: Conn_01x03_Male, Connector_PinHeader_2.54mm:PinHeader_1x03_P2.54mm_Vertical, symbol Connector:Conn_01x03_Male
- added J20: Conn_01x02_Male, Connector_PinHeader_2.54mm:PinHeader_1x02_P2.54mm_Vertical, symbol Connector:Conn_01x02_Male
- added J9: Conn_01x04_Male, PinHeader_1x04_P2.54mm_Vertical, symbol Connector:Conn_01x04_Male
- D10, D2, D3, D4, D5, D6, D7, D8, D9: footprint LED_SMD:LED_PLCC-2 -> splat2-kicad:LED_PLCC-2
- U1: footprint NEO7_GPS_MODULE -> splat2-kicad:NEO7_GPS_MODULE
- U2: footprint ESP-C3-13 -> splat2-kicad:ESP-C3-13
- renumbered J1 to CN11, J2 to CN12
Connections:
- net +3V3: now also J9.1 (Pin_1)
- net +5V: now also J20.2 (Pin_2)
- net 5VEXT: now also J20.1 (Pin_1)
- net GND: now also J9.4 (Pin_4)
- net PB11: now also U6.17 (PB11)
- net PF0: now also J9.3 (Pin_3)
- net PF1: now also J9.2 (Pin_2)
- no-connect marks 70 -> 68
Other:
- note added: "INTERNAL 3V3"
- note added: "INTERNAL 5V"
- note removed: "EXT PWR\nJMPR"
Changed lines of the file:
@@
 F 0 "D7" H 15000 1250 50  0000 C CNN
 F 1 "LED" H 14991 1475 50  0000 C CNN
-F 2 "LED_SMD:LED_PLCC-2" H 15000 1350 50  0001 C CNN
+F 2 "splat2-kicad:LED_PLCC-2" H 15000 1350 50  0001 C CNN
 F 3 "~" H 15000 1350 50  0001 C CNN
 	1    15000 1350
@@
 F 0 "D5" H 14250 1650 50  0000 C CNN
 F 1 "LED" H 14241 1875 50  0000 C CNN
-F 2 "LED_SMD:LED_PLCC-2" H 14250 1750 50  0001 C CNN
+F 2 "splat2-kicad:LED_PLCC-2" H 14250 1750 50  0001 C CNN
 F 3 "~" H 14250 1750 50  0001 C CNN
 	1    14250 1750
@@
 F 0 "D6" H 14650 1450 50  0000 C CNN
 F 1 "LED" H 14641 1675 50  0000 C CNN
-F 2 "LED_SMD:LED_PLCC-2" H 14650 1550 50  0001 C CNN
+F 2 "splat2-kicad:LED_PLCC-2" H 14650 1550 50  0001 C CNN
 F 3 "~" H 14650 1550 50  0001 C CNN
 	1    14650 1550
@@
 F 0 "D4" H 13900 1850 50  0000 C CNN
 F 1 "LED" H 13891 2075 50  0000 C CNN
-F 2 "LED_SMD:LED_PLCC-2" H 13900 1950 50  0001 C CNN
+F 2 "splat2-kicad:LED_PLCC-2" H 13900 1950 50  0001 C CNN
 F 3 "~" H 13900 1950 50  0001 C CNN
 	1    13900 1950
@@
 F 0 "D10" H 15750 1750 50  0000 C CNN
 F 1 "LED" H 15750 2050 50  0000 C CNN
-F 2 "LED_SMD:LED_PLCC-2" H 15750 1900 50  0001 C CNN
+F 2 "splat2-kicad:LED_PLCC-2" H 15750 1900 50  0001 C CNN
 F 3 "~" H 15750 1900 50  0001 C CNN
 	1    15750 1900
@@
 F 0 "D9" H 15742 1054 50  0000 C CNN
 F 1 "LED" H 15742 1145 50  0000 C CNN
-F 2 "LED_SMD:LED_PLCC-2" H 15750 1400 50  0001 C CNN
+F 2 "splat2-kicad:LED_PLCC-2" H 15750 1400 50  0001 C CNN
 F 3 "~" H 15750 1400 50  0001 C CNN
 F 4 "3V3GOOD" H 15742 1236 50  0000 C CNN "DEC"
@@
 F 0 "D3" H 12542 4245 50  0000 C CNN
 F 1 "LED" H 12542 4336 50  0000 C CNN
-F 2 "LED_SMD:LED_PLCC-2" H 12550 4500 50  0001 C CNN
+F 2 "splat2-kicad:LED_PLCC-2" H 12550 4500 50  0001 C CNN
 F 3 "~" H 12550 4500 50  0001 C CNN
 	1    12550 4500
@@
 F 0 "U2" H 5625 8665 50  0000 C CNN
 F 1 "ESP-C3-13U" H 5625 8574 50  0000 C CNN
-F 2 "ESP-C3-13" H 5600 5950 50  0001 C CNN
+F 2 "splat2-kicad:ESP-C3-13" H 5600 5950 50  0001 C CNN
 F 3 "https://docs.ai-thinker.com/_media/esp32/docs/esp-c3-13_specification.pdf" H 3150 5950 50  0001 C CNN
 	1    5600 7250
@@
 Text Label 1150 1300 2    50   ~ 0
 BOOT0
-Text Label 1150 1400 2    50   ~ 0
-PF6
 Text GLabel 1150 1500 0    50   Input ~ 0
 PF7
@@
 GND
 $Comp
-L Connector_Generic:Conn_02x36_Odd_Even J1
+L Connector_Generic:Conn_02x36_Odd_Even CN11
 U 1 1 618B991A
 P 1350 2700
-F 0 "J1" H 1400 4617 50  0000 C CNN
+F 0 "CN11" H 1400 4617 50  0000 C CNN
 F 1 "C11_2X36" H 1400 4526 50  0000 C CNN
 F 2 "Connector_PinSocket_2.54mm:PinSocket_2x36_P2.54mm_Vertical" H 1350 2700 50  0001 C CNN
@@
 Text GLabel 3000 1700 2    50   Input ~ 0
 PB12
-Text Label 3000 1800 0    50   ~ 0
-PB11
 Text GLabel 3000 1900 2    50   Input ~ 0
 GND
@@
 GND
 $Comp
-L Connector_Generic:Conn_02x36_Odd_Even J2
+L Connector_Generic:Conn_02x36_Odd_Even CN12
 U 1 1 61D28094
 P 2700 2700
-F 0 "J2" H 2750 4617 50  0000 C CNN
+F 0 "CN12" H 2750 4617 50  0000 C CNN
 F 1 "C12_2X36" H 2750 4526 50  0000 C CNN
 F 2 "Connector_PinSocket_2.54mm:PinSocket_2x36_P2.54mm_Vertical" H 2700 2700 50  0001 C CNN
@@
 F 0 "U1" H 4150 10778 50  0000 C CNN
 F 1 "ublox_chinese_PCB_module" H 4150 10687 50  0000 C CNN
-F 2 "NEO7_GPS_MODULE" H 4150 10000 50  0001 C CNN
+F 2 "splat2-kicad:NEO7_GPS_MODULE" H 4150 10000 50  0001 C CNN
 F 3 "" H 4150 10100 50  0001 C CNN
 F 4 "M20-7890546" H 4150 10100 50  0001 C CNN "RS Components"
@@
 F 0 "D2" H 7692 6695 50  0000 C CNN
 F 1 "LED" H 7692 6786 50  0000 C CNN
-F 2 "LED_SMD:LED_PLCC-2" H 7700 6950 50  0001 C CNN
+F 2 "splat2-kicad:LED_PLCC-2" H 7700 6950 50  0001 C CNN
 F 3 "~" H 7700 6950 50  0001 C CNN
 	1    7700 6950
@@
 F 0 "D8" H 15542 5795 50  0000 C CNN
 F 1 "LED" H 15542 5886 50  0000 C CNN
-F 2 "LED_SMD:LED_PLCC-2" H 15550 6050 50  0001 C CNN
+F 2 "splat2-kicad:LED_PLCC-2" H 15550 6050 50  0001 C CNN
 F 3 "~" H 15550 6050 50  0001 C CNN
 	1    15550 6050
@@
 Text GLabel 1600 8450 2    50   Input ~ 0
 +3V3
-Text Label 1600 8550 0    50   ~ 0
-PF6
 Text GLabel 1600 8650 2    50   Input ~ 0
 PF7
@@
 Text Notes 750  8600 0    50   ~ 0
 PC_TX
-$Comp
-L Connector:Conn_01x03_Male J9
-U 1 1 630317BA
-P 1150 6500
-F 0 "J9" H 1123 6430 50  0000 R CNN
-F 1 "Conn_01x03_Male" H 1500 6700 50  0000 R CNN
-F 2 "Connector_PinHeader_2.54mm:PinHeader_1x03_P2.54mm_Vertical" H 1150 6500 50  0001 C CNN
-F 3 "~" H 1150 6500 50  0001 C CNN
-F 4 "USER I2C" H 1150 6500 50  0001 C CNN "DESC"
-	1    1150 6500
-	1    0    0    -1
-$EndComp
 Wire Wire Line
 	1350 6400 1550 6400
@@
 Text GLabel 1550 6500 2    50   Input ~ 0
 PF0
-Text Notes 1800 6600 0    50   ~ 0
+Text Notes 1850 6500 0    50   ~ 0
 USER I2C2 BUS\nSCL\nSDA\n
 Wire Wire Line
@@
 NoConn ~ 3000 1500
 NoConn ~ 3000 1600
-NoConn ~ 3000 1800
 NoConn ~ 2500 1700
 NoConn ~ 2500 1600
@@
 NoConn ~ 9950 5400
 NoConn ~ 9950 5500
-NoConn ~ 9950 5700
 NoConn ~ 11950 6300
 NoConn ~ 11950 6200
@@
 	5450 5450 6200 5450
 Wire Wire Line
-	9750 5100 9750 5650
+	9750 5100 9750 5400
 Wire Wire Line
-	3650 5650 9750 5650
+	3650 5650 9200 5650
 Connection ~ 9750 5100
 Wire Wire Line
@@
 Wire Wire Line
 	11400 8900 11500 8900
-Text Notes 11600 8800 0    50   ~ 0
-EXT PWR\nJMPR
+Text Notes 11600 8650 0    50   ~ 0
+INTERNAL 3V3
 Wire Wire Line
 	11500 8900 11500 9000
@@
 Connection ~ 10750 7650
 Wire Wire Line
-	10750 7650 10950 7650
+	10750 7650 10850 7650
 Wire Wire Line
 	9900 7650 9800 7650
@@
 Text GLabel 1150 3800 0    50   Input ~ 0
 PD0
+$Comp
+L Connector:Conn_01x02_Male J20
+U 1 1 61EABEF8
+P 11000 7300
+F 0 "J20" V 11062 7112 50  0000 R CNN
+F 1 "Conn_01x02_Male" V 11153 7112 50  0000 R CNN
+F 2 "Connector_PinHeader_2.54mm:PinHeader_1x02_P2.54mm_Vertical" H 11000 7300 50  0001 C CNN
+F 3 "~" H 11000 7300 50  0001 C CNN
+	1    11000 7300
+	0    -1   1    0
+$EndComp
+Wire Wire Line
+	10850 7650 10850 7500
+Wire Wire Line
+	10850 7500 11000 7500
+Connection ~ 10850 7650
+Wire Wire Line
+	10850 7650 10950 7650
+Wire Wire Line
+	11100 7500 11350 7500
+Wire Wire Line
+	11350 7500 11350 7650
+Wire Wire Line
+	11350 7650 11400 7650
+Text GLabel 11400 7650 2    50   Input ~ 0
++5V
+Text Notes 10800 7300 0    50   ~ 0
+INTERNAL 5V
+$Comp
+L Connector:Conn_01x04_Male J9
+U 1 1 61F8F237
+P 1150 6400
+F 0 "J9" H 1256 6769 50  0000 C CNN
+F 1 "Conn_01x04_Male" H 1256 6678 50  0000 C CNN
+F 2 "PinHeader_1x04_P2.54mm_Vertical" H 1150 6400 50  0001 C CNN
+F 3 "~" H 1150 6400 50  0001 C CNN
+F 4 "I2C2" H 1256 6587 50  0000 C CNN "DESC"
+	1    1150 6400
+	1    0    0    -1
+$EndComp
+Text GLabel 1550 6300 2    50   Input ~ 0
++3V3
+Wire Wire Line
+	1350 6300 1550 6300
+Wire Wire Line
+	9750 5400 9200 5400
+Wire Wire Line
+	9200 5400 9200 5650
+Text GLabel 9700 5700 0    50   Input ~ 0
+PB11
+Text GLabel 3000 1800 2    50   Input ~ 0
+PB11
+Wire Wire Line
+	9950 5700 9700 5700
+Text GLabel 1600 8550 2    50   Input ~ 0
+PF6
+Text GLabel 1150 1400 0    50   Input ~ 0
+PF6
 $EndSCHEMATC

Commit message: Sent off for PCB manufacture
Connections:
- net PF5 is gone; now on net GND: CN12.36 (Pin_36)
- no-connect marks 68 -> 67
Other:
- note added: "3V3 Regulator"
- note added: "VER 0.20 13-Jan-22\nStart Splat2 Rev A: Fixes from prototype PCB"
- note removed: "3V3 Regulator - 5A ???"
- note removed: "VER 0.20\nStart Splat2 Rev A: Fixes from prototype PCB"
Changed lines of the file:
@@
 $EndComp
 Connection ~ 4300 10900
-$Comp
-L Connector:TestPoint TP13
-U 1 1 5C43FB2E
-P 15700 9450
-F 0 "TP13" H 15758 9570 50  0000 L CNN
-F 1 "TestPoint" H 15758 9479 50  0000 L CNN
-F 2 "TestPoint:TestPoint_Loop_D1.80mm_Drill1.0mm_Beaded" H 15900 9450 50  0001 C CNN
-F 3 "~" H 15900 9450 50  0001 C CNN
-	1    15700 9450
-	-1   0    0    -1
-$EndComp
 Wire Wire Line
 	10100 10750 10100 11050
@@
 SERIAL FLASH ROM\n  AND NVRAM
 Text Notes 12400 10400 0    89   Italic 0
-VER 0.20\nStart Splat2 Rev A: Fixes from prototype PCB
+VER 0.20  13-Jan-22\nStart Splat2 Rev A: Fixes from prototype PCB
 $Comp
 L Connector_Generic:Conn_01x02 J14
@@
 Wire Wire Line
 	10950 11000 11050 11000
-Text Notes 10650 8450 0    50   ~ 0
-3V3 Regulator - 5A ???
+Text Notes 10900 8550 0    50   ~ 0
+3V3 Regulator
 $Comp
 L Connector:Screw_Terminal_01x02 J17
@@
 NoConn ~ 3000 3000
 NoConn ~ 3000 2800
-NoConn ~ 3000 2700
 NoConn ~ 3000 2300
 NoConn ~ 3000 2400
@@
 Text Label 3000 2600 0    50   ~ 0
 PC4
-Text Label 3000 2700 0    50   ~ 0
-PF5
 Text Label 3000 2800 0    50   ~ 0
 PF4
@@
 Text GLabel 1150 1400 0    50   Input ~ 0
 PF6
+Text GLabel 3000 2700 2    50   Input ~ 0
+PF5
+Text GLabel 3950 3650 2    50   Input ~ 0
+PF5
+Wire Wire Line
+	3950 3650 3850 3650
+Wire Wire Line
+	3850 3650 3850 3800
+Connection ~ 3850 3800
+$Comp
+L Connector:TestPoint TP13
+U 1 1 5C43FB2E
+P 15700 9450
+F 0 "TP13" H 15758 9570 50  0000 L CNN
+F 1 "TestPoint" H 15758 9479 50  0000 L CNN
+F 2 "TestPoint:TestPoint_Loop_D1.80mm_Drill1.0mm_Beaded" H 15900 9450 50  0001 C CNN
+F 3 "~" H 15900 9450 50  0001 C CNN
+	1    15700 9450
+	-1   0    0    -1
+$EndComp
 $EndSCHEMATC
